Commit message: Fix mesh inclusion in URDF for proper display in Gazebo

File: pizibot_description/urdf/lidar.xacro (robot description, xacro)
@@ -10,5 +10,5 @@
             <origin xyz="0 0 -${lidar_origin_height_offset}" rpy="0 0 0"/>
             <geometry>
-                <mesh filename="package://pizibot_description/meshes/lidar_with_support.stl" scale="0.001 0.001 0.001"/>
+                <mesh filename="file://$(find pizibot_description)/meshes/lidar_with_support.stl" scale="0.001 0.001 0.001"/>
             </geometry>
             <material name="gray"/>

File: pizibot_description/urdf/pizibot_macro.xacro (robot description, xacro)
@@ -20,5 +20,5 @@
             <visual>
                 <geometry>
-                    <mesh filename="package://pizibot_description/meshes/chassis.stl" scale="0.001 0.001 0.001"/>
+                    <mesh filename="file://$(find pizibot_description)/meshes/chassis.stl" scale="0.001 0.001 0.001"/>
                 </geometry>
                 <material name="white"/>
@@ -26,5 +26,5 @@
             <collision>
                 <geometry>
-                    <mesh filename="package://pizibot_description/meshes/chassis.stl" scale="0.001 0.001 0.001"/>
+                    <mesh filename="file://$(find pizibot_description)/meshes/chassis.stl" scale="0.001 0.001 0.001"/>
                 </geometry>
             </collision>
@@ -46,5 +46,5 @@
             <visual>
                 <geometry>
-                    <mesh filename="package://pizibot_description/meshes/left_wheel.stl" scale="0.001 0.001 0.001"/>
+                    <mesh filename="file://$(find pizibot_description)/meshes/left_wheel.stl" scale="0.001 0.001 0.001"/>
                 </geometry>
                 <material name="red"/>
@@ -72,5 +72,5 @@
             <visual>
                 <geometry>
-                    <mesh filename="package://pizibot_description/meshes/right_wheel.stl" scale="0.001 0.001 0.001"/>
+                    <mesh filename="file://$(find pizibot_description)/meshes/right_wheel.stl" scale="0.001 0.001 0.001"/>
                 </geometry>
                 <material name="red"/>

Commit message: Preparation of description file separation for simulation and real robot

File: pizibot_description/urdf/lidar.xacro (robot description, xacro)
@@ -27,5 +27,5 @@
     <gazebo reference="$(arg prefix)laser_frame">
         <material>Gazebo/Black</material>
-        <sensor name="laser" type="ray">
+        <sensor name="$(arg prefix)laser" type="ray">
             <pose>0 0 0 0 0 0</pose>        <!-- Position and orientation of the sensor -->
             <visualize>false</visualize>    <!-- Set to true to visualize the lidar in Gazebo -->
@@ -44,7 +44,7 @@
                 </range>
             </ray>
-            <plugin name="laser_controller" filename="libgazebo_ros_ray_sensor.so"> <!-- Plugin for ROS integration -->
+            <plugin name="$(arg prefix)laser_controller" filename="libgazebo_ros_ray_sensor.so"> <!-- Plugin for ROS integration -->
                 <ros>
-                    <argument>~/out:=scan</argument> <!-- ROS topic for lidar output -->
+                    <argument>~/out:=$(arg prefix)scan</argument> <!-- ROS topic for lidar output -->
                 </ros>
                 <output_type>sensor_msgs/LaserScan</output_type> <!-- Type of output message -->

File: pizibot_description/urdf/pizibot_macro.xacro (robot description, xacro)
@@ -15,5 +15,5 @@
             <parent link="${prefix}base_link"/>
             <child link="${prefix}chassis"/>
-            <origin xyz="0 0 0" rpy="0 0 0"/>
+            <origin xyz="0 0 0" rpy="0 0 -${pi/2}"/>
         </joint>
         <link name="${prefix}chassis">
