Commit message: Update mesh access method based on simulation vs. real robot environment. - Use <xacro:if> for absolute path access (file://) in simulation mode.

File: pizibot_description/urdf/camera.xacro (robot description, xacro)
@@ -10,5 +10,10 @@
             <origin xyz="0 0 0" rpy="0 0 0"/>
             <geometry>
-                <mesh filename="file://$(find pizibot_description)/meshes/camera_support.stl" scale="0.001 0.001 0.001"/>
+                <xacro:if value="$(arg sim_mode)">
+                    <mesh filename="file://$(find pizibot_description)/meshes/camera_support.stl" scale="0.001 0.001 0.001"/>
+                </xacro:if >
+                <xacro:unless value="$(arg sim_mode)">
+                    <!-- TODO -->
+                </xacro:unless>
             </geometry>
             <material name="gray"/>
@@ -17,5 +22,10 @@
             <origin xyz="0 0 0" rpy="0 0 0"/>
             <geometry>
-                <mesh filename="file://$(find pizibot_description)/meshes/camera_support.stl" scale="0.001 0.001 0.001"/>
+                <xacro:if value="$(arg sim_mode)">
+                    <mesh filename="file://$(find pizibot_description)/meshes/camera_support.stl" scale="0.001 0.001 0.001"/>
+                </xacro:if >
+                <xacro:unless value="$(arg sim_mode)">
+                    <!-- TODO -->
+                </xacro:unless>
             </geometry>
         </collision>
@@ -28,11 +38,17 @@
     <link name="$(arg prefix)camera_link">
         <visual>
-            <origin xyz="-0.009 0 -0.011" rpy="${pi/2} 0 ${pi/2}"/> <!-- Value to align the camera visual in the correct direction and set the origin at the lens -->
+            <origin xyz="-0.009 0 -0.011" rpy="${pi/2} 0 ${pi/2}"/>
+            <!-- Value to align the camera visual in the correct direction and set the origin at the lens -->
             <geometry>
-                <mesh filename="file://$(find pizibot_description)/meshes/esp_cam.stl" scale="0.001 0.001 0.001"/>
+                <xacro:if value="$(arg sim_mode)">
+                    <mesh filename="file://$(find pizibot_description)/meshes/esp_cam.stl" scale="0.001 0.001 0.001"/>
+                </xacro:if >
+                <xacro:unless value="$(arg sim_mode)">
+                    <!-- TODO -->
+                </xacro:unless>
             </geometry>
             <material name="red"/>
         </visual>
-            <!-- No collision as the camera is inside the support -->
+        <!-- No collision as the camera is inside the support -->
     </link>
     <joint name="$(arg prefix)camera_optical_joint" type="fixed">
@@ -47,10 +63,10 @@
             <pose> 0 0 0 0 0 0 </pose>
             <visualize>true</visualize>
-            <update_rate>15</update_rate> <!-- Max frame rate at full resolution -->
+            <update_rate>15</update_rate>            <!-- Max frame rate at full resolution -->
             <camera>
                 <horizontal_fov>1.089</horizontal_fov>
                 <image>
                     <format>RGB8</format>
-                    <width>1600</width> <!-- UXGA resolution -->
+                    <width>1600</width>                    <!-- UXGA resolution -->
                     <height>1200</height>
                 </image>

File: pizibot_description/urdf/lidar.xacro (robot description, xacro)
@@ -10,5 +10,10 @@
             <origin xyz="0 0 -${lidar_origin_height_offset}" rpy="0 0 0"/>
             <geometry>
-                <mesh filename="file://$(find pizibot_description)/meshes/lidar_with_support.stl" scale="0.001 0.001 0.001"/>
+                <xacro:if value="$(arg sim_mode)">
+                    <mesh filename="file://$(find pizibot_description)/meshes/lidar_with_support.stl" scale="0.001 0.001 0.001"/>
+                </xacro:if >
+                <xacro:unless value="$(arg sim_mode)">
+                    <!-- TODO -->
+                </xacro:unless>
             </geometry>
             <material name="gray"/>
@@ -24,10 +29,10 @@
         </xacro:inertial_cylinder>
     </link>
-     <!-- Gazebo specific settings for the lidar -->
+    <!-- Gazebo specific settings for the lidar -->
     <gazebo reference="$(arg prefix)laser_frame">
         <material>Gazebo/Black</material>
         <sensor name="$(arg prefix)laser" type="ray">
-            <pose>0 0 0 0 0 0</pose>        <!-- Position and orientation of the sensor -->
-            <visualize>false</visualize>    <!-- Set to true to visualize the lidar in Gazebo -->
+            <pose>0 0 0 0 0 0</pose>            <!-- Position and orientation of the sensor -->
+            <visualize>false</visualize>            <!-- Set to true to visualize the lidar in Gazebo -->
             <update_rate>10</update_rate>
             <ray>
@@ -44,10 +49,10 @@
                 </range>
             </ray>
-            <plugin name="$(arg prefix)laser_controller" filename="libgazebo_ros_ray_sensor.so"> <!-- Plugin for ROS integration -->
+            <plugin name="$(arg prefix)laser_controller" filename="libgazebo_ros_ray_sensor.so">                <!-- Plugin for ROS integration -->
                 <ros>
-                    <argument>~/out:=$(arg prefix)scan</argument> <!-- ROS topic for lidar output -->
+                    <argument>~/out:=$(arg prefix)scan</argument>                    <!-- ROS topic for lidar output -->
                 </ros>
-                <output_type>sensor_msgs/LaserScan</output_type> <!-- Type of output message -->
-                <frame_name>$(arg prefix)laser_frame</frame_name>               <!-- Frame name for the sensor -->
+                <output_type>sensor_msgs/LaserScan</output_type>                <!-- Type of output message -->
+                <frame_name>$(arg prefix)laser_frame</frame_name>                <!-- Frame name for the sensor -->
             </plugin>
         </sensor>

File: pizibot_description/urdf/pizibot_macro.xacro (robot description, xacro)
@@ -21,5 +21,10 @@
                 <origin xyz="0 0 0" rpy="0 0 ${pi}"/>
                 <geometry>
-                    <mesh filename="file://$(find pizibot_description)/meshes/chassis.stl" scale="0.001 0.001 0.001"/>
+                    <xacro:if value="$(arg sim_mode)">
+                        <mesh filename="file://$(find pizibot_description)/meshes/chassis.stl" scale="0.001 0.001 0.001"/>
+                    </xacro:if >
+                    <xacro:unless value="$(arg sim_mode)">
+                        <!-- TODO -->
+                    </xacro:unless>
                 </geometry>
                 <material name="white"/>
@@ -49,5 +54,10 @@
                 <origin xyz="0 0 0" rpy="0 ${pi} 0"/>
                 <geometry>
-                    <mesh filename="file://$(find pizibot_description)/meshes/left_wheel.stl" scale="0.001 0.001 0.001"/>
+                    <xacro:if value="$(arg sim_mode)">
+                        <mesh filename="file://$(find pizibot_description)/meshes/left_wheel.stl" scale="0.001 0.001 0.001"/>
+                    </xacro:if >
+                    <xacro:unless value="$(arg sim_mode)">
+                        <!-- TODO -->
+                    </xacro:unless>
                 </geometry>
                 <material name="red"/>
@@ -75,5 +85,10 @@
             <visual>
                 <geometry>
-                    <mesh filename="file://$(find pizibot_description)/meshes/right_wheel.stl" scale="0.001 0.001 0.001"/>
+                    <xacro:if value="$(arg sim_mode)">
+                        <mesh filename="file://$(find pizibot_description)/meshes/right_wheel.stl" scale="0.001 0.001 0.001"/>
+                    </xacro:if >
+                    <xacro:unless value="$(arg sim_mode)">
+                        <!-- TODO -->
+                    </xacro:unless>
                 </geometry>
                 <material name="red"/>

Commit message: Update mesh access method for simulation and real robot environments.
- Implement `xacro:unless` to use package-based paths (package://) for the real robot.

File: pizibot_description/urdf/camera.xacro (robot description, xacro)
@@ -14,5 +14,5 @@
                 </xacro:if >
                 <xacro:unless value="$(arg sim_mode)">
-                    <!-- TODO -->
+                        <mesh filename="package://pizibot_description/meshes/camera_support.stl" scale="0.001 0.001 0.001"/>
                 </xacro:unless>
             </geometry>
@@ -26,5 +26,5 @@
                 </xacro:if >
                 <xacro:unless value="$(arg sim_mode)">
-                    <!-- TODO -->
+                        <mesh filename="package://pizibot_description/meshes/camera_support.stl" scale="0.001 0.001 0.001"/>
                 </xacro:unless>
             </geometry>
@@ -45,5 +45,5 @@
                 </xacro:if >
                 <xacro:unless value="$(arg sim_mode)">
-                    <!-- TODO -->
+                        <mesh filename="package://pizibot_description/meshes/esp_cam.stl" scale="0.001 0.001 0.001"/>
                 </xacro:unless>
             </geometry>

File: pizibot_description/urdf/lidar.xacro (robot description, xacro)
@@ -14,5 +14,5 @@
                 </xacro:if >
                 <xacro:unless value="$(arg sim_mode)">
-                    <!-- TODO -->
+                        <mesh filename="package://pizibot_description/meshes/lidar_with_support.stl" scale="0.001 0.001 0.001"/>
                 </xacro:unless>
             </geometry>

File: pizibot_description/urdf/pizibot_macro.xacro (robot description, xacro)
@@ -25,5 +25,5 @@
                     </xacro:if >
                     <xacro:unless value="$(arg sim_mode)">
-                        <!-- TODO -->
+                        <mesh filename="package://pizibot_description/meshes/chassis.stl" scale="0.001 0.001 0.001"/>
                     </xacro:unless>
                 </geometry>
@@ -58,5 +58,5 @@
                     </xacro:if >
                     <xacro:unless value="$(arg sim_mode)">
-                        <!-- TODO -->
+                        <mesh filename="package://pizibot_description/meshes/left_wheel.stl" scale="0.001 0.001 0.001"/>
                     </xacro:unless>
                 </geometry>
@@ -89,5 +89,5 @@
                     </xacro:if >
                     <xacro:unless value="$(arg sim_mode)">
-                        <!-- TODO -->
+                        <mesh filename="package://pizibot_description/meshes/right_wheel.stl" scale="0.001 0.001 0.001"/>
                     </xacro:unless>
                 </geometry>
