Commit message: Refactor Pizibot robot description for ROS 2 Jazzy compatibility
- Added README.md to provide an overview of the Pizibot robot description package, including usage instructions and package structure.
- Updated rsp.launch.py to remove the prefix argument and streamline robot identification.
- Modified RViz configuration to reflect changes in robot link names and improve visualization settings.
- Refactored camera.xacro to remove prefix arguments and simplify mesh loading logic.
- Introduced control.xacro for hardware control configuration, replacing the deprecated ros2_control.xacro.
- Added gazebo_config.xacro for Gazebo-specific settings, enhancing simulation integration.
- Updated lidar.xacro to improve sensor configuration and remove unnecessary prefix arguments.
- Refined dimensions.xacro to include additional properties for camera and lidar settings.
- Updated pizibot.urdf.xacro and pizibot_macro.xacro to remove prefix arguments and ensure consistency across robot components.

File: pizibot_description/urdf/camera.xacro (robot description, xacro)
@@ -1,19 +1,14 @@
 <?xml version="1.0"?>
 <robot xmlns:xacro="http://www.ros.org/wiki/xacro">
-    <joint name="$(arg prefix)camera_support_joint" type="fixed">
-        <parent link="$(arg prefix)chassis"/>
-        <child link="$(arg prefix)camera_support_link"/>
+    <joint name="camera_support_joint" type="fixed">
+        <parent link="chassis"/>
+        <child link="camera_support_link"/>
         <origin xyz="0 0 0" rpy="0 0 ${pi}"/>
     </joint>
-    <link name="$(arg prefix)camera_support_link">
+    <link name="camera_support_link">
         <visual>
             <origin xyz="0 0 0" rpy="0 0 0"/>
             <geometry>
-                <xacro:if value="$(arg sim_mode)">
-                    <mesh filename="file://$(find pizibot_description)/meshes/camera_support.stl" scale="0.001 0.001 0.001"/>
-                </xacro:if >
-                <xacro:unless value="$(arg sim_mode)">
-                        <mesh filename="package://pizibot_description/meshes/camera_support.stl" scale="0.001 0.001 0.001"/>
-                </xacro:unless>
+                <mesh filename="package://pizibot_description/meshes/camera_support.stl" scale="0.001 0.001 0.001"/>
             </geometry>
             <material name="gray"/>
@@ -22,29 +17,19 @@
             <origin xyz="0 0 0" rpy="0 0 0"/>
             <geometry>
-                <xacro:if value="$(arg sim_mode)">
-                    <mesh filename="file://$(find pizibot_description)/meshes/camera_support.stl" scale="0.001 0.001 0.001"/>
-                </xacro:if >
-                <xacro:unless value="$(arg sim_mode)">
-                        <mesh filename="package://pizibot_description/meshes/camera_support.stl" scale="0.001 0.001 0.001"/>
-                </xacro:unless>
+                <mesh filename="package://pizibot_description/meshes/camera_support.stl" scale="0.001 0.001 0.001"/>
             </geometry>
         </collision>
     </link>
-    <joint name="$(arg prefix)camera_joint" type="fixed">
-        <parent link="$(arg prefix)chassis"/>
-        <child link="$(arg prefix)camera_link"/>
+    <joint name="camera_joint" type="fixed">
+        <parent link="chassis"/>
+        <child link="camera_link"/>
         <origin xyz="0 ${camera_distance} ${camera_base_height}" rpy="0 0 ${pi/2}"/>
     </joint>
-    <link name="$(arg prefix)camera_link">
+    <link name="camera_link">
         <visual>
             <origin xyz="-0.009 0 -0.011" rpy="${pi/2} 0 ${pi/2}"/>
             <!-- Value to align the camera visual in the correct direction and set the origin at the lens -->
             <geometry>
-                <xacro:if value="$(arg sim_mode)">
-                    <mesh filename="file://$(find pizibot_description)/meshes/esp_cam.stl" scale="0.001 0.001 0.001"/>
-                </xacro:if >
-                <xacro:unless value="$(arg sim_mode)">
-                        <mesh filename="package://pizibot_description/meshes/esp_cam.stl" scale="0.001 0.001 0.001"/>
-                </xacro:unless>
+                <mesh filename="package://pizibot_description/meshes/esp_cam.stl" scale="0.001 0.001 0.001"/>
             </geometry>
             <material name="red"/>
@@ -52,31 +37,31 @@
         <!-- No collision as the camera is inside the support -->
     </link>
-    <joint name="$(arg prefix)camera_optical_joint" type="fixed">
+    <joint name="camera_optical_joint" type="fixed">
         <origin xyz="0 0 0" rpy="${-pi/2} 0 ${-pi/2}" />
-        <parent link="$(arg prefix)camera_link" />
-        <child link="$(arg prefix)camera_link_optical" />
+        <parent link="camera_link" />
+        <child link="camera_link_optical" />
     </joint>
-    <link name="$(arg prefix)camera_link_optical"></link>
-    <gazebo reference="$(arg prefix)camera_link">
+    <link name="camera_link_optical"></link>
+    <gazebo reference="camera_link">
         <material>Gazebo/Red</material>
-        <sensor name="$(arg prefix)camera" type="camera">
-            <pose> 0 0 0 0 0 0 </pose>
+        <sensor name="camera" type="camera">
+            <pose>0 0 0 0 0 0</pose>
             <visualize>true</visualize>
-            <update_rate>15</update_rate>            <!-- Max frame rate at full resolution -->
+            <update_rate>${camera_update_rate}</update_rate>
             <camera>
-                <horizontal_fov>1.089</horizontal_fov>
+                <horizontal_fov>${camera_horizontal_fov}</horizontal_fov>
                 <image>
-                    <format>RGB8</format>
-                    <width>1600</width>                    <!-- UXGA resolution -->
-                    <height>1200</height>
+                    <format>R8G8B8</format>
+                    <width>${camera_width}</width>
+                    <height>${camera_height}</height>
                 </image>
                 <clip>
-                    <near>0.05</near>
-                    <far>8.0</far>
+                    <near>${camera_clip_near}</near>
+                    <far>${camera_clip_far}</far>
                 </clip>
             </camera>
-            <plugin name="$(arg prefix)camera_controller" filename="libgazebo_ros_camera.so">
-                <frame_name>$(arg prefix)camera_link_optical</frame_name>
-            </plugin>
+            <topic>camera/image_raw</topic>
+            <camera_info_topic>camera/camera_info</camera_info_topic>
+            <gz_frame_id>camera_link_optical</gz_frame_id>
         </sensor>
     </gazebo>

File: pizibot_description/urdf/dimensions.xacro (robot description, xacro)
@@ -8,4 +8,9 @@
     <xacro:property name="wheel_diameter" value="0.08" />
     <xacro:property name="wheel_mass" value="0.1" />
+    <xacro:property name="wheel_separation" value="0.273" />
+    <!-- Max wheel velocity property in rad/s (125 RPM ≈ 13.09 rad/s) -->
+    <xacro:property name="max_wheel_velocity" value="13.09" />
+    <!-- Max wheel effort in Nm -->
+    <xacro:property name="max_wheel_effort" value="40" />
     <xacro:property name="ground_clearance" value="0.018" />
     <xacro:property name="caster_wheel_distance" value="0.120" />
@@ -14,11 +19,20 @@
     <!-- RPLIDAR A1M8 properties -->
     <xacro:property name="lidar_distance" value="0.084" /> <!-- Distance from chassis origin to lidar origin on X axis -->
-    <xacro:property name="lidar_diameter" value="0.098" />   <!-- support_lidar length  -->
+    <xacro:property name="lidar_diameter" value="0.098" /> <!-- support_lidar length -->
     <xacro:property name="lidar_length" value="0.062" /> <!-- lidar height + lidar support height -->
-    <xacro:property name="lidar_height" value="0.115" />
     <xacro:property name="lidar_origin_height_offset" value="0.007" /> <!-- the frame origin is at 7 mm from the top of the lidar -->
-    <xacro:property name="lidar_mass" value="0.0" />  <!-- 0 because his mass is include in the robot mass -->
-    <!-- camera -->
+    <xacro:property name="lidar_mass" value="0.0" /> <!-- 0 because his mass is included in the robot mass -->
+    <xacro:property name="lidar_update_rate" value="10" />
+    <xacro:property name="lidar_samples" value="360" />
+    <xacro:property name="lidar_min_range" value="0.15" />
+    <xacro:property name="lidar_max_range" value="12.0" />
+    <!-- Camera properties -->
     <xacro:property name="camera_base_height" value="0.097" />
     <xacro:property name="camera_distance" value="0.194" />
+    <xacro:property name="camera_update_rate" value="15" />
+    <xacro:property name="camera_horizontal_fov" value="1.089" />
+    <xacro:property name="camera_width" value="1600" />
+    <xacro:property name="camera_height" value="1200" />
+    <xacro:property name="camera_clip_near" value="0.05" />
+    <xacro:property name="camera_clip_far" value="8.0" />
 </robot>

File: pizibot_description/urdf/lidar.xacro (robot description, xacro)
@@ -1,19 +1,14 @@
 <?xml version="1.0"?>
 <robot xmlns:xacro="http://www.ros.org/wiki/xacro">
-    <joint name="$(arg prefix)laser_joint" type="fixed">
-        <parent link="$(arg prefix)chassis"/>
-        <child link="$(arg prefix)laser_frame"/>
+    <joint name="laser_joint" type="fixed">
+        <parent link="chassis"/>
+        <child link="laser_frame"/>
         <origin xyz="0 ${lidar_distance} ${robot_height+lidar_length}" rpy="0 0 ${3*pi/2}"/>
     </joint>
-    <link name="$(arg prefix)laser_frame">
+    <link name="laser_frame">
         <visual>
             <origin xyz="0 0 -${lidar_origin_height_offset}" rpy="0 0 0"/>
             <geometry>
-                <xacro:if value="$(arg sim_mode)">
-                    <mesh filename="file://$(find pizibot_description)/meshes/lidar_with_support.stl" scale="0.001 0.001 0.001"/>
-                </xacro:if >
-                <xacro:unless value="$(arg sim_mode)">
-                        <mesh filename="package://pizibot_description/meshes/lidar_with_support.stl" scale="0.001 0.001 0.001"/>
-                </xacro:unless>
+                <mesh filename="package://pizibot_description/meshes/lidar_with_support.stl" scale="0.001 0.001 0.001"/>
             </geometry>
             <material name="gray"/>
@@ -30,30 +25,26 @@
     </link>
     <!-- Gazebo specific settings for the lidar -->
-    <gazebo reference="$(arg prefix)laser_frame">
+    <gazebo reference="laser_frame">
         <material>Gazebo/Black</material>
-        <sensor name="$(arg prefix)laser" type="ray">
-            <pose>0 0 0 0 0 0</pose>            <!-- Position and orientation of the sensor -->
-            <visualize>false</visualize>            <!-- Set to true to visualize the lidar in Gazebo -->
-            <update_rate>10</update_rate>
-            <ray>
+        <sensor name="laser" type="gpu_lidar">
+            <always_on>true</always_on>
+            <pose>0 0 0 0 0 0</pose>
+            <visualize>true</visualize>
+            <update_rate>${lidar_update_rate}</update_rate>
+            <lidar>
                 <scan>
                     <horizontal>
-                        <samples>360</samples>
-                        <min_angle>-3.14</min_angle>
-                        <max_angle>3.14</max_angle>
+                        <samples>${lidar_samples}</samples>
+                        <min_angle>-${pi}</min_angle>
+                        <max_angle>${pi}</max_angle>
                     </horizontal>
                 </scan>
                 <range>
-                    <min>0.15</min>
-                    <max>12.0</max>
+                    <min>${lidar_min_range}</min>
+                    <max>${lidar_max_range}</max>
                 </range>
-            </ray>
-            <plugin name="$(arg prefix)laser_controller" filename="libgazebo_ros_ray_sensor.so">                <!-- Plugin for ROS integration -->
-                <ros>
-                    <argument>~/out:=$(arg prefix)scan</argument>                    <!-- ROS topic for lidar output -->
-                </ros>
-                <output_type>sensor_msgs/LaserScan</output_type>                <!-- Type of output message -->
-                <frame_name>$(arg prefix)laser_frame</frame_name>                <!-- Frame name for the sensor -->
-            </plugin>
+            </lidar>
+            <topic>scan</topic>
+            <gz_frame_id>laser_frame</gz_frame_id>
         </sensor>
     </gazebo>

File: pizibot_description/urdf/pizibot.urdf.xacro (robot description, xacro)
@@ -1,5 +1,5 @@
 <?xml version="1.0"?>
 <robot xmlns:xacro="http://www.ros.org/wiki/xacro" name="pizibot">
-    <xacro:arg name="prefix" default=""/>
+    <!-- prefix removed: names are unprefixed now -->
     <xacro:arg name="sim_mode" default="false"/>
     <xacro:include filename="material_colors.xacro" />
@@ -8,6 +8,6 @@
     <xacro:include filename="pizibot_macro.xacro" />
     <xacro:include filename="lidar.xacro" />
-    <xacro:include filename="ros2_control.xacro" />
+    <xacro:include filename="control.xacro" />
     <xacro:include filename="camera.xacro" />
-    <xacro:pizibot prefix="$(arg prefix)"/>
+    <xacro:pizibot/>
 </robot>

File: pizibot_description/urdf/pizibot_macro.xacro (robot description, xacro)
@@ -1,30 +1,25 @@
 <?xml version="1.0"?>
 <robot xmlns:xacro="http://www.ros.org/wiki/xacro">
-    <xacro:macro name="pizibot" params="prefix">
+    <xacro:macro name="pizibot">
         <!-- BASE LINK -->
-        <link name="${prefix}base_link"></link>
+        <link name="base_link"></link>
         <!-- BASE LINK FOOTPRINT -->
-        <link name="${prefix}base_footprint"></link>
-        <joint name="${prefix}base_footprint_joint" type="fixed">
-            <parent link="${prefix}base_link"/>
-            <child link="${prefix}base_footprint"/>
+        <link name="base_footprint"></link>
+        <joint name="base_footprint_joint" type="fixed">
+            <parent link="base_link"/>
+            <child link="base_footprint"/>
             <origin xyz="0 0 -${ground_clearance/2}" rpy="0 0 0"/>
         </joint>
         <!-- CHASSIS -->
-        <joint name="${prefix}chassis_joint" type="fixed">
-            <parent link="${prefix}base_link"/>
-            <child link="${prefix}chassis"/>
+        <joint name="chassis_joint" type="fixed">
+            <parent link="base_link"/>
+            <child link="chassis"/>
             <origin xyz="0 0 0" rpy="0 0 -${pi/2}"/>
         </joint>
-        <link name="${prefix}chassis">
+        <link name="chassis">
             <visual>
                 <origin xyz="0 0 0" rpy="0 0 ${pi}"/>
                 <geometry>
-                    <xacro:if value="$(arg sim_mode)">
-                        <mesh filename="file://$(find pizibot_description)/meshes/chassis.stl" scale="0.001 0.001 0.001"/>
-                    </xacro:if >
-                    <xacro:unless value="$(arg sim_mode)">
-                        <mesh filename="package://pizibot_description/meshes/chassis.stl" scale="0.001 0.001 0.001"/>
-                    </xacro:unless>
+                    <mesh filename="package://pizibot_description/meshes/chassis.stl" scale="0.001 0.001 0.001"/>
                 </geometry>
                 <material name="white"/>
@@ -40,24 +35,20 @@
             </xacro:inertial_cylinder>
         </link>
-        <gazebo reference="${prefix}chassis">
+        <gazebo reference="chassis">
             <material>Gazebo/SkyBlue</material>
         </gazebo>
         <!-- left_wheel -->
-        <joint name="${prefix}left_wheel_joint" type="continuous">
-            <parent link="${prefix}chassis"/>
-            <child link="${prefix}left_wheel"/>
+        <joint name="left_wheel_joint" type="continuous">
+            <parent link="chassis"/>
+            <child link="left_wheel"/>
             <origin xyz="${-((robot_diameter/2)-(wheel_width/2))} 0 ${ground_clearance}" rpy="-${pi/2} 0 ${pi/2}"/>
             <axis xyz="0 0 1"/>
+            <limit effort="${max_wheel_effort}" velocity="${max_wheel_velocity}"/>
         </joint>
-        <link name="${prefix}left_wheel">
+        <link name="left_wheel">
             <visual>
                 <origin xyz="0 0 0" rpy="0 ${pi} 0"/>
                 <geometry>
-                    <xacro:if value="$(arg sim_mode)">
-                        <mesh filename="file://$(find pizibot_description)/meshes/left_wheel.stl" scale="0.001 0.001 0.001"/>
-                    </xacro:if >
-                    <xacro:unless value="$(arg sim_mode)">
-                        <mesh filename="package://pizibot_description/meshes/left_wheel.stl" scale="0.001 0.001 0.001"/>
-                    </xacro:unless>
+                    <mesh filename="package://pizibot_description/meshes/left_wheel.stl" scale="0.001 0.001 0.001"/>
                 </geometry>
                 <material name="red"/>
@@ -72,23 +63,19 @@
             </xacro:inertial_cylinder>
         </link>
-        <gazebo reference="${prefix}left_wheel">
+        <gazebo reference="left_wheel">
             <material>Gazebo/Red</material>
         </gazebo>
         <!-- right_wheel -->
-        <joint name="${prefix}right_wheel_joint" type="continuous">
-            <parent link="${prefix}chassis"/>
-            <child link="${prefix}right_wheel"/>
+        <joint name="right_wheel_joint" type="continuous">
+            <parent link="chassis"/>
+            <child link="right_wheel"/>
             <origin xyz="${((robot_diameter/2)-(wheel_width/2))} 0 ${ground_clearance}" rpy="-${pi/2} 0 -${pi/2}"/>
             <axis xyz="0 0 -1"/>
+            <limit effort="${max_wheel_effort}" velocity="${max_wheel_velocity}"/>
         </joint>
-        <link name="${prefix}right_wheel">
+        <link name="right_wheel">
             <visual>
                 <geometry>
-                    <xacro:if value="$(arg sim_mode)">
-                        <mesh filename="file://$(find pizibot_description)/meshes/right_wheel.stl" scale="0.001 0.001 0.001"/>
-                    </xacro:if >
-                    <xacro:unless value="$(arg sim_mode)">
-                        <mesh filename="package://pizibot_description/meshes/right_wheel.stl" scale="0.001 0.001 0.001"/>
-                    </xacro:unless>
+                    <mesh filename="package://pizibot_description/meshes/right_wheel.stl" scale="0.001 0.001 0.001"/>
                 </geometry>
                 <material name="red"/>
@@ -103,14 +90,14 @@
             </xacro:inertial_cylinder>
         </link>
-        <gazebo reference="${prefix}right_wheel">
+        <gazebo reference="right_wheel">
             <material>Gazebo/Red</material>
         </gazebo>
         <!-- FRONT CASTER WHEEL -->
-        <joint name="$(arg prefix)front_caster_wheel_joint" type="fixed">
-            <parent link="${prefix}chassis"/>
-            <child link="$(arg prefix)front_caster_wheel"/>
+        <joint name="front_caster_wheel_joint" type="fixed">
+            <parent link="chassis"/>
+            <child link="front_caster_wheel"/>
             <origin xyz="0 -${caster_wheel_distance} 0" rpy="0 0 0"/>
         </joint>
-        <link name="$(arg prefix)front_caster_wheel">
+        <link name="front_caster_wheel">
             <visual>
                 <geometry>
@@ -128,5 +115,5 @@
             </xacro:inertial_sphere>
         </link>
-        <gazebo reference="$(arg prefix)front_caster_wheel">
+        <gazebo reference="front_caster_wheel">
             <material>Gazebo/Black</material>
             <mu1 value="0.001"/>
@@ -134,10 +121,10 @@
         </gazebo>
         <!-- BACK CASTER WHEEL -->
-        <joint name="$(arg prefix)back_caster_wheel_joint" type="fixed">
-            <parent link="${prefix}chassis"/>
-            <child link="$(arg prefix)back_caster_wheel"/>
+        <joint name="back_caster_wheel_joint" type="fixed">
+            <parent link="chassis"/>
+            <child link="back_caster_wheel"/>
             <origin xyz="0 ${caster_wheel_distance} 0" rpy="0 0 0"/>
         </joint>
-        <link name="$(arg prefix)back_caster_wheel">
+        <link name="back_caster_wheel">
             <visual>
                 <geometry>
@@ -155,5 +142,5 @@
             </xacro:inertial_sphere>
         </link>
-        <gazebo reference="$(arg prefix)front_caster_wheel">
+        <gazebo reference="back_caster_wheel">
             <material>Gazebo/Black</material>
             <mu1 value="0.001"/>
