Commit message: Refactor URDF and RViz configurations for Pizibot V2
- Removed obsolete STL files: camera_support.stl, chassis.stl, esp_cam.stl, left_wheel.stl, right_wheel.stl.
- Added new STL files: robot_chassis.stl, rplidar_a1.stl, tire_80mm.stl, wheel.stl.
- Updated camera.xacro to remove camera support link and adjust camera joint parameters.
- Modified control.xacro to update wheel parameters for improved performance.
- Adjusted dimensions.xacro to reflect new robot dimensions and properties.
- Enhanced lidar.xacro to include visual representation for the RPLIDAR.
- Updated pizibot_macro.xacro to replace chassis visual with new robot chassis model and adjust wheel links.
- Revised RViz configuration files to reflect changes in link names for caster wheels.
- Updated hardware parameters in README and YAML files to match new specifications.
- Adjusted navigation parameters to match new specifications.

File: pizibot_description/urdf/camera.xacro (robot description, xacro)
@@ -1,39 +1,10 @@
 <?xml version="1.0"?>
 <robot xmlns:xacro="http://www.ros.org/wiki/xacro">
-    <joint name="camera_support_joint" type="fixed">
-        <parent link="chassis"/>
-        <child link="camera_support_link"/>
-        <origin xyz="0 0 0" rpy="0 0 ${pi}"/>
-    </joint>
-    <link name="camera_support_link">
-        <visual>
-            <origin xyz="0 0 0" rpy="0 0 0"/>
-            <geometry>
-                <mesh filename="package://pizibot_description/meshes/camera_support.stl" scale="0.001 0.001 0.001"/>
-            </geometry>
-            <material name="gray"/>
-        </visual>
-        <collision>
-            <origin xyz="0 0 0" rpy="0 0 0"/>
-            <geometry>
-                <mesh filename="package://pizibot_description/meshes/camera_support.stl" scale="0.001 0.001 0.001"/>
-            </geometry>
-        </collision>
-    </link>
     <joint name="camera_joint" type="fixed">
         <parent link="chassis"/>
         <child link="camera_link"/>
-        <origin xyz="0 ${camera_distance} ${camera_base_height}" rpy="0 0 ${pi/2}"/>
+        <origin xyz="0 ${camera_x_offset} ${camera_z_offset}" rpy="0 0 ${pi/2}"/>
     </joint>
     <link name="camera_link">
-        <visual>
-            <origin xyz="-0.009 0 -0.011" rpy="${pi/2} 0 ${pi/2}"/>
-            <!-- Value to align the camera visual in the correct direction and set the origin at the lens -->
-            <geometry>
-                <mesh filename="package://pizibot_description/meshes/esp_cam.stl" scale="0.001 0.001 0.001"/>
-            </geometry>
-            <material name="red"/>
-        </visual>
-        <!-- No collision as the camera is inside the support -->
     </link>
     <joint name="camera_optical_joint" type="fixed">
@@ -53,6 +24,6 @@
                 <image>
                     <format>R8G8B8</format>
-                    <width>${camera_width}</width>
-                    <height>${camera_height}</height>
+                    <width>${camera_image_width}</width>
+                    <height>${camera_image_height}</height>
                 </image>
                 <clip>
@@ -77,6 +48,6 @@
                 <horizontal_fov>${camera_horizontal_fov}</horizontal_fov>
                 <image>
-                    <width>${camera_width}</width>
-                    <height>${camera_height}</height>
+                    <width>${camera_image_width}</width>
+                    <height>${camera_image_height}</height>
                 </image>
                 <clip>

File: pizibot_description/urdf/control.xacro (robot description, xacro)
@@ -3,5 +3,5 @@
     <!-- Gazebo Harmonic simulation  -->
     <xacro:if value="$(arg sim_mode)">
-        <xacro:include filename="gazebo_config.xacro" />
+        <xacro:include filename="$(find pizibot_description)/urdf/gazebo_config.xacro" />
     </xacro:if>
     <!-- Real hardware control block -->
@@ -13,6 +13,6 @@
                 <param name="baud_rate">115200</param>
                 <param name="encoder_ppr">1320</param>
-                <param name="wheel_radius">0.033</param>
-                <param name="wheel_separation">0.17</param>
+                <param name="wheel_radius">0.04</param>
+                <param name="wheel_separation">0.29</param>
             </hardware>
             <joint name="left_wheel_joint">

File: pizibot_description/urdf/dimensions.xacro (robot description, xacro)
@@ -2,25 +2,29 @@
 <robot xmlns:xacro="http://ros.org/wiki/xacro">
     <!-- Robot property -->
-    <xacro:property name="robot_diameter" value="0.300" />
-    <xacro:property name="robot_height" value="0.108" />
+    <xacro:property name="robot_diameter" value="0.290" />
+    <!-- with wheel  -->
+    <xacro:property name="robot_height" value="0.103" />
     <xacro:property name="robot_mass" value="1" />
-    <xacro:property name="wheel_width" value="0.027" />
+    <xacro:property name="wheel_width" value="0.04" />
     <xacro:property name="wheel_diameter" value="0.08" />
     <xacro:property name="wheel_mass" value="0.1" />
-    <xacro:property name="wheel_separation" value="0.273" />
-    <!-- Max wheel velocity property in rad/s (125 RPM ≈ 13.09 rad/s) -->
-    <xacro:property name="max_wheel_velocity" value="13.09" />
+    <xacro:property name="wheel_separation" value="0.29" />
+    <xacro:property name="wheel_y_offset" value="0.01969" />
+    <!-- Max wheel velocity property in rad/s (4.6 rad/s RPM ≈ 43.93 RPM) -->
+    <xacro:property name="max_wheel_velocity" value="4.6" />
     <!-- Max wheel effort in Nm -->
     <xacro:property name="max_wheel_effort" value="40" />
-    <xacro:property name="ground_clearance" value="0.018" />
-    <xacro:property name="caster_wheel_distance" value="0.120" />
-    <xacro:property name="caster_wheel_diameter" value="${0.007+ground_clearance*2}" />
-    <xacro:property name="caster_wheel_mass" value="0.1" />
+    <xacro:property name="ground_clearance" value="${0.057-(caster_diameter/2)}" />
+    <xacro:property name="caster_x_offset" value="0.09" />
+    <xacro:property name="caster_diameter" value="0.016" />
+    <xacro:property name="caster_mass" value="0.1" />
     <!-- RPLIDAR A1M8 properties -->
-    <xacro:property name="lidar_distance" value="0.084" /> <!-- Distance from chassis origin to lidar origin on X axis -->
-    <xacro:property name="lidar_diameter" value="0.098" /> <!-- support_lidar length -->
-    <xacro:property name="lidar_length" value="0.062" /> <!-- lidar height + lidar support height -->
-    <xacro:property name="lidar_origin_height_offset" value="0.007" /> <!-- the frame origin is at 7 mm from the top of the lidar -->
-    <xacro:property name="lidar_mass" value="0.0" /> <!-- 0 because his mass is included in the robot mass -->
+    <xacro:property name="lidar_x_offset" value="0.055" />
+    <!-- Distance from chassis origin to lidar origin on X axis -->
+    <xacro:property name="lidar_diameter" value="0.098" />
+    <!-- support_lidar length -->
+    <xacro:property name="lidar_height" value="0.062" />
+    <!-- lidar height + lidar support height -->
+    <xacro:property name="lidar_mass" value="0.1" />
     <xacro:property name="lidar_update_rate" value="10" />
     <xacro:property name="lidar_samples" value="360" />
@@ -28,10 +32,10 @@
     <xacro:property name="lidar_max_range" value="12.0" />
     <!-- Camera properties -->
-    <xacro:property name="camera_base_height" value="0.097" />
-    <xacro:property name="camera_distance" value="0.194" />
+    <xacro:property name="camera_z_offset" value="0.080" />
+    <xacro:property name="camera_x_offset" value="${robot_diameter/2}" />
     <xacro:property name="camera_update_rate" value="15" />
     <xacro:property name="camera_horizontal_fov" value="1.089" />
-    <xacro:property name="camera_width" value="1600" />
-    <xacro:property name="camera_height" value="1200" />
+    <xacro:property name="camera_image_width" value="1600" />
+    <xacro:property name="camera_image_height" value="1200" />
     <xacro:property name="camera_clip_near" value="0.05" />
     <xacro:property name="camera_clip_far" value="8.0" />

File: pizibot_description/urdf/lidar.xacro (robot description, xacro)
@@ -4,23 +4,30 @@
         <parent link="chassis"/>
         <child link="laser_frame"/>
-        <origin xyz="0 ${lidar_distance} ${robot_height+lidar_length}" rpy="0 0 ${3*pi/2}"/>
+        <origin xyz="0 -${lidar_x_offset} ${robot_height+lidar_height}" rpy="0 0 ${pi/2}"/>
     </joint>
     <link name="laser_frame">
+        <collision>
+            <origin xyz="0 0 -${lidar_height/2}" rpy="0 0 0"/>
+            <geometry>
+                <cylinder radius="${lidar_diameter/2}" length="${lidar_height}"/>
+            </geometry>
+        </collision>
+        <xacro:inertial_cylinder mass="${lidar_mass}" length="${lidar_height}" radius="${lidar_diameter/2}">
+            <origin xyz="0 0 -${lidar_height/2}" rpy="0 0 0"/>
+        </xacro:inertial_cylinder>
+    </link>
+    <joint name="laser_visual_joint" type="fixed">
+        <parent link="chassis"/>
+        <child link="laser_visual"/>
+        <origin xyz="0 0 0" rpy="${pi/2} 0 ${pi}"/>
+    </joint>
+    <link name="laser_visual">
         <visual>
-            <origin xyz="0 0 -${lidar_origin_height_offset}" rpy="0 0 0"/>
+            <origin xyz="0 0 0" rpy="0 0 0"/>
             <geometry>
-                <mesh filename="package://pizibot_description/meshes/lidar_with_support.stl" scale="0.001 0.001 0.001"/>
+                <mesh filename="package://pizibot_description/meshes/rplidar_a1.stl" scale="0.001 0.001 0.001"/>
             </geometry>
             <material name="gray"/>
         </visual>
-        <collision>
-            <origin xyz="0 0 -${lidar_length/2}" rpy="0 0 0"/>
-            <geometry>
-                <cylinder radius="${lidar_diameter/2}" length="${lidar_length}"/>
-            </geometry>
-        </collision>
-        <xacro:inertial_cylinder mass="${lidar_mass}" length="${lidar_length}" radius="${lidar_diameter/2}">
-            <origin xyz="0 0 0" rpy="0 0 0"/>
-        </xacro:inertial_cylinder>
     </link>
     <!-- Gazebo specific settings for the lidar -->

File: pizibot_description/urdf/pizibot.urdf.xacro (robot description, xacro)
@@ -3,11 +3,11 @@
     <!-- prefix removed: names are unprefixed now -->
     <xacro:arg name="sim_mode" default="false"/>
-    <xacro:include filename="material_colors.xacro" />
-    <xacro:include filename="inertial_macros.xacro" />
-    <xacro:include filename="dimensions.xacro" />
-    <xacro:include filename="pizibot_macro.xacro" />
-    <xacro:include filename="lidar.xacro" />
-    <xacro:include filename="control.xacro" />
-    <xacro:include filename="camera.xacro" />
+    <xacro:include filename="$(find pizibot_description)/urdf/material_colors.xacro" />
+    <xacro:include filename="$(find pizibot_description)/urdf/inertial_macros.xacro" />
+    <xacro:include filename="$(find pizibot_description)/urdf/dimensions.xacro" />
+    <xacro:include filename="$(find pizibot_description)/urdf/pizibot_macro.xacro" />
+    <xacro:include filename="$(find pizibot_description)/urdf/lidar.xacro" />
+    <xacro:include filename="$(find pizibot_description)/urdf/control.xacro" />
+    <xacro:include filename="$(find pizibot_description)/urdf/camera.xacro" />
     <xacro:pizibot/>
 </robot>

File: pizibot_description/urdf/pizibot_macro.xacro (robot description, xacro)
@@ -18,11 +18,4 @@
         </joint>
         <link name="chassis">
-            <visual>
-                <origin xyz="0 0 0" rpy="0 0 ${pi}"/>
-                <geometry>
-                    <mesh filename="package://pizibot_description/meshes/chassis.stl" scale="0.001 0.001 0.001"/>
-                </geometry>
-                <material name="white"/>
-            </visual>
             <collision>
                 <origin xyz="0 0 ${robot_height/2}" rpy="0 0 0"/>
@@ -32,9 +25,23 @@
             </collision>
             <xacro:inertial_cylinder mass="${robot_mass}" length="${robot_height}" radius="${robot_diameter/2}">
-                <origin xyz="${robot_diameter/2} 0 ${robot_height/2}" rpy="0 0 0"/>
+                <origin xyz="0 0 ${robot_height/2}" rpy="0 0 0"/>
             </xacro:inertial_cylinder>
         </link>
-        <gazebo reference="chassis">
-            <material>Gazebo/SkyBlue</material>
+        <joint name="chassis_visual_joint" type="fixed">
+            <parent link="base_link"/>
+            <child link="chassis_visual"/>
+            <origin xyz="0 0 0" rpy="${pi/2} 0 ${pi/2}"/>
+        </joint>
+        <link name="chassis_visual">
+            <visual>
+                <origin xyz="0 0 0" rpy="0 0 0 "/>
+                <geometry>
+                    <mesh filename="package://pizibot_description/meshes/robot_chassis.stl" scale="0.001 0.001 0.001"/>
+                </geometry>
+                <material name="white"/>
+            </visual>
+        </link>
+        <gazebo reference="chassis_visual">
+            <material>Gazebo/White</material>
         </gazebo>
         <!-- left_wheel -->
@@ -42,5 +49,5 @@
             <parent link="chassis"/>
             <child link="left_wheel"/>
-            <origin xyz="${-((robot_diameter/2)-(wheel_width/2))} 0 ${ground_clearance}" rpy="-${pi/2} 0 ${pi/2}"/>
+            <origin xyz="${-((robot_diameter/2)-(wheel_width/2))} 0 -${wheel_y_offset}" rpy="-${pi/2} 0 ${pi/2}"/>
             <axis xyz="0 0 1"/>
             <limit effort="${max_wheel_effort}" velocity="${max_wheel_velocity}"/>
@@ -48,7 +55,7 @@
         <link name="left_wheel">
             <visual>
-                <origin xyz="0 0 0" rpy="0 ${pi} 0"/>
+                <origin xyz="0 0 0" rpy="0 0 0"/>
                 <geometry>
-                    <mesh filename="package://pizibot_description/meshes/left_wheel.stl" scale="0.001 0.001 0.001"/>
+                    <mesh filename="package://pizibot_description/meshes/wheel.stl" scale="0.001 0.001 0.001"/>
                 </geometry>
                 <material name="red"/>
@@ -70,5 +77,5 @@
             <parent link="chassis"/>
             <child link="right_wheel"/>
-            <origin xyz="${((robot_diameter/2)-(wheel_width/2))} 0 ${ground_clearance}" rpy="-${pi/2} 0 -${pi/2}"/>
+            <origin xyz="${((robot_diameter/2)-(wheel_width/2))} 0 -${wheel_y_offset}" rpy="-${pi/2} 0 -${pi/2}"/>
             <axis xyz="0 0 -1"/>
             <limit effort="${max_wheel_effort}" velocity="${max_wheel_velocity}"/>
@@ -77,5 +84,5 @@
             <visual>
                 <geometry>
-                    <mesh filename="package://pizibot_description/meshes/right_wheel.stl" scale="0.001 0.001 0.001"/>
+                    <mesh filename="package://pizibot_description/meshes/wheel.stl" scale="0.001 0.001 0.001"/>
                 </geometry>
                 <material name="red"/>
@@ -94,13 +101,13 @@
         </gazebo>
         <!-- FRONT CASTER WHEEL -->
-        <joint name="front_caster_wheel_joint" type="fixed">
+        <joint name="front_caster_joint" type="fixed">
             <parent link="chassis"/>
-            <child link="front_caster_wheel"/>
-            <origin xyz="0 -${caster_wheel_distance} 0" rpy="0 0 0"/>
+            <child link="front_caster"/>
+            <origin xyz="0 ${caster_x_offset} -${ground_clearance}" rpy="0 0 0"/>
         </joint>
-        <link name="front_caster_wheel">
+        <link name="front_caster">
             <visual>
                 <geometry>
-                    <sphere radius="${caster_wheel_diameter/2}" />
+                    <sphere radius="${caster_diameter/2}" />
                 </geometry>
                 <material name="black"/>
@@ -108,12 +115,12 @@
             <collision>
                 <geometry>
-                    <sphere radius="${caster_wheel_diameter/2}" />
+                    <sphere radius="${caster_diameter/2}" />
                 </geometry>
             </collision>
-            <xacro:inertial_sphere mass="${caster_wheel_mass}" radius="${caster_wheel_diameter/2}">
+            <xacro:inertial_sphere mass="${caster_mass}" radius="${caster_diameter/2}">
                 <origin xyz="0 0 0" rpy="0 0 0"/>
             </xacro:inertial_sphere>
         </link>
-        <gazebo reference="front_caster_wheel">
+        <gazebo reference="front_caster">
             <material>Gazebo/Black</material>
             <mu1 value="0.001"/>
@@ -121,13 +128,13 @@
         </gazebo>
         <!-- BACK CASTER WHEEL -->
-        <joint name="back_caster_wheel_joint" type="fixed">
+        <joint name="back_caster_joint" type="fixed">
             <parent link="chassis"/>
-            <child link="back_caster_wheel"/>
-            <origin xyz="0 ${caster_wheel_distance} 0" rpy="0 0 0"/>
+            <child link="back_caster"/>
+            <origin xyz="0 -${caster_x_offset} -${ground_clearance}" rpy="0 0 0"/>
         </joint>
-        <link name="back_caster_wheel">
+        <link name="back_caster">
             <visual>
                 <geometry>
-                    <sphere radius="${caster_wheel_diameter/2}" />
+                    <sphere radius="${caster_diameter/2}" />
                 </geometry>
                 <material name="black"/>
@@ -135,16 +142,44 @@
             <collision>
                 <geometry>
-                    <sphere radius="${caster_wheel_diameter/2}" />
+                    <sphere radius="${caster_diameter/2}" />
                 </geometry>
             </collision>
-            <xacro:inertial_sphere mass="${caster_wheel_mass}" radius="${caster_wheel_diameter/2}">
+            <xacro:inertial_sphere mass="${caster_mass}" radius="${caster_diameter/2}">
                 <origin xyz="0 0 0" rpy="0 0 0"/>
             </xacro:inertial_sphere>
         </link>
-        <gazebo reference="back_caster_wheel">
+        <gazebo reference="back_caster">
             <material>Gazebo/Black</material>
             <mu1 value="0.001"/>
             <mu2 value="0.001"/>
         </gazebo>
+        <!-- FRONT CASTER CYLINDER -->
+        <joint name="front_caster_cylinder_joint" type="fixed">
+            <parent link="chassis"/>
+            <child link="front_caster_cylinder"/>
+            <origin xyz="0 ${caster_x_offset} 0" rpy="0 0 0"/>
+        </joint>
+        <link name="front_caster_cylinder">
+            <collision>
+                <origin xyz="0 0 -${ground_clearance/2}" rpy="0 0 0 "/>
+                <geometry>
+                    <cylinder length="${ground_clearance}" radius="${caster_diameter/2}" />
+                </geometry>
+            </collision>
+        </link>
+        <!-- BACK CASTER CYLINDER -->
+        <joint name="back_caster_cylinder_joint" type="fixed">
+            <parent link="chassis"/>
+            <child link="back_caster_cylinder"/>
+            <origin xyz="0 -${caster_x_offset} 0" rpy="0 0 0"/>
+        </joint>
+        <link name="back_caster_cylinder">
+            <collision>
+                <origin xyz="0 0 -${ground_clearance/2}" rpy="0 0 0 "/>
+                <geometry>
+                    <cylinder length="${ground_clearance}" radius="${caster_diameter/2}" />
+                </geometry>
+            </collision>
+        </link>
     </xacro:macro>
 </robot>
