Commit message: fix(description,hardware): derive control params from xacro and add wheel friction
- control.xacro: read wheel_radius/wheel_separation from
  dimensions.xacro instead of hardcoding; fix encoder_ppr (1320 -> 330)
- pizibot_macro.xacro: fix base_footprint origin (use full
  ground_clearance instead of half); add mu1/mu2 wheel friction
- dimensions.xacro: add wheel_friction property, reorder
  ground_clearance after caster_diameter definition
- robot_controllers.yaml: update odometry covariances to measured
  values; disable enable_odom_tf (EKF now publishes odom->base_link)
- Update pizibot_hardware README

File: pizibot_description/urdf/control.xacro (robot description, xacro)
@@ -12,7 +12,7 @@
                 <param name="serial_port">/dev/ttyESP32</param>
                 <param name="baud_rate">115200</param>
-                <param name="encoder_ppr">1320</param>
-                <param name="wheel_radius">0.04</param>
-                <param name="wheel_separation">0.29</param>
+                <param name="encoder_ppr">330</param>
+                <param name="wheel_radius">${wheel_diameter/2}</param>
+                <param name="wheel_separation">${wheel_separation}</param>
             </hardware>
             <joint name="left_wheel_joint">

File: pizibot_description/urdf/pizibot_macro.xacro (robot description, xacro)
@@ -9,5 +9,5 @@
             <parent link="base_link"/>
             <child link="base_footprint"/>
-            <origin xyz="0 0 -${ground_clearance/2}" rpy="0 0 0"/>
+            <origin xyz="0 0 -${ground_clearance}" rpy="0 0 0"/>
         </joint>
         <!-- CHASSIS -->
@@ -35,5 +35,5 @@
         <link name="chassis_visual">
             <visual>
-                <origin xyz="0 0 0" rpy="0 0 0 "/>
+                <origin xyz="0 0 0" rpy="0 0 0"/>
                 <geometry>
                     <mesh filename="package://pizibot_description/meshes/robot_chassis.stl" scale="0.001 0.001 0.001"/>
@@ -72,4 +72,6 @@
         <gazebo reference="left_wheel">
             <material>Gazebo/Red</material>
+            <mu1 value="${wheel_friction}"/>
+            <mu2 value="${wheel_friction}"/>
         </gazebo>
         <!-- right_wheel -->
@@ -99,4 +101,6 @@
         <gazebo reference="right_wheel">
             <material>Gazebo/Red</material>
+            <mu1 value="${wheel_friction}"/>
+            <mu2 value="${wheel_friction}"/>
         </gazebo>
         <!-- FRONT CASTER WHEEL -->
@@ -162,5 +166,5 @@
         <link name="front_caster_cylinder">
             <collision>
-                <origin xyz="0 0 -${ground_clearance/2}" rpy="0 0 0 "/>
+                <origin xyz="0 0 -${ground_clearance/2}" rpy="0 0 0"/>
                 <geometry>
                     <cylinder length="${ground_clearance}" radius="${caster_diameter/2}" />
@@ -176,5 +180,5 @@
         <link name="back_caster_cylinder">
             <collision>
-                <origin xyz="0 0 -${ground_clearance/2}" rpy="0 0 0 "/>
+                <origin xyz="0 0 -${ground_clearance/2}" rpy="0 0 0"/>
                 <geometry>
                     <cylinder length="${ground_clearance}" radius="${caster_diameter/2}" />
