Commit message: Adding lidar description

File: pizibot_description/urdf/dimensions.xacro (robot description, xacro)
@@ -1,5 +1,5 @@
 <?xml version="1.0" ?>
 <robot xmlns:xacro="http://ros.org/wiki/xacro">
-    <!-- PROPERTY -->
+    <!-- Robot property -->
     <xacro:property name="robot_diameter" value="0.300" />
     <xacro:property name="robot_height" value="0.108" />
@@ -12,3 +12,10 @@
     <xacro:property name="caster_wheel_diameter" value="${ground_clearance*2}" />
     <xacro:property name="caster_wheel_mass" value="0.1" />
+    <!-- RPLIDAR A1M8 properties -->
+    <xacro:property name="lidar_distance" value="0.084" /> <!-- Distance from chassis origin to lidar origin on X axis -->
+    <xacro:property name="lidar_diameter" value="0.098" />   <!-- support_lidar length  -->
+    <xacro:property name="lidar_length" value="0.062" /> <!-- lidar height + lidar support height -->
+    <xacro:property name="lidar_height" value="0.115" />
+    <xacro:property name="lidar_origin_height_offset" value="0.007" /> <!-- the frame origin is at 7 mm from the top of the lidar -->
+    <xacro:property name="lidar_mass" value="0.3" />
 </robot>

File: pizibot_description/urdf/material_colors.xacro (robot description, xacro)
@@ -16,3 +16,9 @@
         <color rgba="0 0 0 1"/>
     </material>
+    <material name="gray">
+        <color rgba="0.5 0.5 0.5 1"/>
+    </material>
+    <material name="light_blue">
+        <color rgba="0.678 0.847 0.902 1"/>
+    </material>
 </robot>

File: pizibot_description/urdf/pizibot.urdf.xacro (robot description, xacro)
@@ -1,4 +1,4 @@
 <?xml version="1.0"?>
-<robot xmlns:xacro="http://www.ros.org/wiki/xacro"  name="pizibot">
+<robot xmlns:xacro="http://www.ros.org/wiki/xacro" name="pizibot">
     <xacro:arg name="prefix" default=""/>
     <xacro:include filename="material_colors.xacro" />
@@ -6,4 +6,5 @@
     <xacro:include filename="dimensions.xacro" />
     <xacro:include filename="pizibot_macro.xacro" />
+    <xacro:include filename="lidar.xacro" />
     <xacro:pizibot prefix="$(arg prefix)"/>
 </robot>

Commit message: Preparing description packge for simulation

File: pizibot_description/urdf/dimensions.xacro (robot description, xacro)
@@ -18,4 +18,4 @@
     <xacro:property name="lidar_height" value="0.115" />
     <xacro:property name="lidar_origin_height_offset" value="0.007" /> <!-- the frame origin is at 7 mm from the top of the lidar -->
-    <xacro:property name="lidar_mass" value="0.3" />
+    <xacro:property name="lidar_mass" value="0.0" />  <!-- 0 because his mass is include in the robot mass -->
 </robot>

File: pizibot_description/urdf/lidar.xacro (robot description, xacro)
@@ -4,5 +4,5 @@
         <parent link="$(arg prefix)chassis"/>
         <child link="$(arg prefix)laser_frame"/>
-        <origin xyz="0 -${lidar_distance} ${robot_height+lidar_length}" rpy="0 0 ${3*pi/2}"/>
+        <origin xyz="0 ${lidar_distance} ${robot_height+lidar_length}" rpy="0 0 ${3*pi/2}"/>
     </joint>
     <link name="$(arg prefix)laser_frame">
@@ -49,5 +49,5 @@
                 </ros>
                 <output_type>sensor_msgs/LaserScan</output_type> <!-- Type of output message -->
-                <frame_name>laser_frame</frame_name>               <!-- Frame name for the sensor -->
+                <frame_name>$(arg prefix)laser_frame</frame_name>               <!-- Frame name for the sensor -->
             </plugin>
         </sensor>

File: pizibot_description/urdf/pizibot.urdf.xacro (robot description, xacro)
@@ -2,4 +2,5 @@
 <robot xmlns:xacro="http://www.ros.org/wiki/xacro" name="pizibot">
     <xacro:arg name="prefix" default=""/>
+    <xacro:arg name="sim_mode" default="false"/>
     <xacro:include filename="material_colors.xacro" />
     <xacro:include filename="inertial_macros.xacro" />

File: pizibot_description/urdf/pizibot_macro.xacro (robot description, xacro)
@@ -15,8 +15,9 @@
             <parent link="${prefix}base_link"/>
             <child link="${prefix}chassis"/>
-            <origin xyz="0 0 0" rpy="0 0 ${pi/2}"/>
+            <origin xyz="0 0 0" rpy="0 0 0"/>
         </joint>
         <link name="${prefix}chassis">
             <visual>
+                <origin xyz="0 0 0" rpy="0 0 ${pi}"/>
                 <geometry>
                     <mesh filename="file://$(find pizibot_description)/meshes/chassis.stl" scale="0.001 0.001 0.001"/>
@@ -25,6 +26,7 @@
             </visual>
             <collision>
+                <origin xyz="0 0 ${robot_height/2}" rpy="0 0 0"/>
                 <geometry>
-                    <mesh filename="file://$(find pizibot_description)/meshes/chassis.stl" scale="0.001 0.001 0.001"/>
+                    <cylinder length="${robot_height}" radius="${robot_diameter/2}" />
                 </geometry>
             </collision>
@@ -40,9 +42,10 @@
             <parent link="${prefix}chassis"/>
             <child link="${prefix}left_wheel"/>
-            <origin xyz="${-((robot_diameter/2)-(wheel_width/2))} 0 ${ground_clearance}" rpy="-${pi/2} 0 -${pi/2}"/>
+            <origin xyz="${-((robot_diameter/2)-(wheel_width/2))} 0 ${ground_clearance}" rpy="-${pi/2} 0 ${pi/2}"/>
             <axis xyz="0 0 1"/>
         </joint>
         <link name="${prefix}left_wheel">
             <visual>
+                <origin xyz="0 0 0" rpy="0 ${pi} 0"/>
                 <geometry>
                     <mesh filename="file://$(find pizibot_description)/meshes/left_wheel.stl" scale="0.001 0.001 0.001"/>

Commit message: Add camera description and rviz config for simulation

File: pizibot_description/urdf/dimensions.xacro (robot description, xacro)
@@ -10,5 +10,5 @@
     <xacro:property name="ground_clearance" value="0.018" />
     <xacro:property name="caster_wheel_distance" value="0.120" />
-    <xacro:property name="caster_wheel_diameter" value="${ground_clearance*2}" />
+    <xacro:property name="caster_wheel_diameter" value="${0.007+ground_clearance*2}" />
     <xacro:property name="caster_wheel_mass" value="0.1" />
     <!-- RPLIDAR A1M8 properties -->
@@ -19,3 +19,6 @@
     <xacro:property name="lidar_origin_height_offset" value="0.007" /> <!-- the frame origin is at 7 mm from the top of the lidar -->
     <xacro:property name="lidar_mass" value="0.0" />  <!-- 0 because his mass is include in the robot mass -->
+    <!-- camera -->
+    <xacro:property name="camera_base_height" value="0.097" />
+    <xacro:property name="camera_distance" value="0.194" />
 </robot>

File: pizibot_description/urdf/pizibot.urdf.xacro (robot description, xacro)
@@ -9,4 +9,5 @@
     <xacro:include filename="lidar.xacro" />
     <xacro:include filename="ros2_control.xacro" />
+    <xacro:include filename="camera.xacro" />
     <xacro:pizibot prefix="$(arg prefix)"/>
 </robot>

Commit message: feat(description,navigation): add IMU sensor and fuse it via EKF
- Add imu.xacro defining imu_link, joint (with offsets), and the
  Gazebo IMU sensor plugin
- Include imu.xacro from pizibot.urdf.xacro
- Remove IMU sensor and /tf topic remap from gazebo_config.xacro
  (moved to imu.xacro)
- Add imu_x/y/z_offset properties to dimensions.xacro
- ekf.yaml: fuse only IMU angular velocity (yaw), not absolute
  orientation, since imu_link is yaw-rotated relative to base_link;
  disable gravity removal (real IMU has no orientation quaternion);
  fuse only vx from odom; remove map_frame; add transform_timeout
- Launch the EKF node from online_async_launch.py (mapping) in
  addition to localization_launch.py
- Update pizibot_description

File: pizibot_description/urdf/dimensions.xacro (robot description, xacro)
@@ -11,12 +11,13 @@
     <xacro:property name="wheel_separation" value="0.29" />
     <xacro:property name="wheel_y_offset" value="0.01969" />
+    <xacro:property name="wheel_friction" value="1.0" />
     <!-- Max wheel velocity property in rad/s (4.6 rad/s RPM ≈ 43.93 RPM) -->
     <xacro:property name="max_wheel_velocity" value="4.6" />
     <!-- Max wheel effort in Nm -->
     <xacro:property name="max_wheel_effort" value="40" />
-    <xacro:property name="ground_clearance" value="${0.057-(caster_diameter/2)}" />
     <xacro:property name="caster_x_offset" value="0.09" />
     <xacro:property name="caster_diameter" value="0.016" />
     <xacro:property name="caster_mass" value="0.1" />
+    <xacro:property name="ground_clearance" value="${0.057-(caster_diameter/2)}" />
     <!-- RPLIDAR A1M8 properties -->
     <xacro:property name="lidar_x_offset" value="0.055" />
@@ -40,3 +41,7 @@
     <xacro:property name="camera_clip_near" value="0.05" />
     <xacro:property name="camera_clip_far" value="8.0" />
+    <!-- IMU properties -->
+    <xacro:property name="imu_x_offset" value="-0.011" />
+    <xacro:property name="imu_y_offset" value="0.100" />
+    <xacro:property name="imu_z_offset" value="0.092" />
 </robot>

File: pizibot_description/urdf/gazebo_config.xacro (robot description, xacro)
@@ -21,5 +21,4 @@
             <frame_id>odom</frame_id>
             <child_frame_id>base_link</child_frame_id>
-            <tf_topic>/tf</tf_topic>
             <odom_publisher_frequency>50</odom_publisher_frequency>
         </plugin>
@@ -29,57 +28,4 @@
             <joint_name>right_wheel_joint</joint_name>
         </plugin>
-        <plugin filename="gz-sim-imu-system" name="gz::sim::systems::Imu">
-        </plugin>
-    </gazebo>
-    <!-- IMU Sensor -->
-    <gazebo reference="base_link">
-        <sensor name="imu_sensor" type="imu">
-            <always_on>true</always_on>
-            <update_rate>100</update_rate>
-            <topic>imu</topic>
-            <gz_frame_id>base_link</gz_frame_id>
-            <imu>
-                <angular_velocity>
-                    <x>
-                        <noise type="gaussian">
-                            <mean>0.0</mean>
-                            <stddev>0.0002</stddev>
-                        </noise>
-                    </x>
-                    <y>
-                        <noise type="gaussian">
-                            <mean>0.0</mean>
-                            <stddev>0.0002</stddev>
-                        </noise>
-                    </y>
-                    <z>
-                        <noise type="gaussian">
-                            <mean>0.0</mean>
-                            <stddev>0.0002</stddev>
-                        </noise>
-                    </z>
-                </angular_velocity>
-                <linear_acceleration>
-                    <x>
-                        <noise type="gaussian">
-                            <mean>0.0</mean>
-                            <stddev>0.017</stddev>
-                        </noise>
-                    </x>
-                    <y>
-                        <noise type="gaussian">
-                            <mean>0.0</mean>
-                            <stddev>0.017</stddev>
-                        </noise>
-                    </y>
-                    <z>
-                        <noise type="gaussian">
-                            <mean>0.0</mean>
-                            <stddev>0.017</stddev>
-                        </noise>
-                    </z>
-                </linear_acceleration>
-            </imu>
-        </sensor>
     </gazebo>
 </robot>

File: pizibot_description/urdf/pizibot.urdf.xacro (robot description, xacro)
@@ -10,4 +10,5 @@
     <xacro:include filename="$(find pizibot_description)/urdf/control.xacro" />
     <xacro:include filename="$(find pizibot_description)/urdf/camera.xacro" />
+    <xacro:include filename="$(find pizibot_description)/urdf/imu.xacro" />
     <xacro:pizibot/>
 </robot>

Commit message: fix: update wheel separation and max velocity parameters for consistency

File: pizibot_description/urdf/dimensions.xacro (robot description, xacro)
@@ -9,9 +9,9 @@
     <xacro:property name="wheel_diameter" value="0.08" />
     <xacro:property name="wheel_mass" value="0.1" />
-    <xacro:property name="wheel_separation" value="0.29" />
+    <xacro:property name="wheel_separation" value="0.26" />
     <xacro:property name="wheel_y_offset" value="0.01969" />
     <xacro:property name="wheel_friction" value="1.0" />
-    <!-- Max wheel velocity property in rad/s (4.6 rad/s RPM ≈ 43.93 RPM) -->
-    <xacro:property name="max_wheel_velocity" value="4.6" />
+    <!-- Max wheel velocity property in rad/s (13.0 rad/s ≈ 124.1 RPM, matches WHEEL_CMD_MAX_RADS) -->
+    <xacro:property name="max_wheel_velocity" value="13.0" />
     <!-- Max wheel effort in Nm -->
     <xacro:property name="max_wheel_effort" value="40" />

File: pizibot_description/urdf/gazebo_config.xacro (robot description, xacro)
@@ -13,8 +13,8 @@
             <wheel_separation>${wheel_separation}</wheel_separation>
             <wheel_radius>${wheel_diameter/2}</wheel_radius>
-            <max_linear_acceleration>1.0</max_linear_acceleration>
-            <min_linear_acceleration>-1.0</min_linear_acceleration>
-            <max_angular_acceleration>2.0</max_angular_acceleration>
-            <min_angular_acceleration>-2.0</min_angular_acceleration>
+            <max_linear_acceleration>2.0</max_linear_acceleration>
+            <min_linear_acceleration>-2.0</min_linear_acceleration>
+            <max_angular_acceleration>1.8</max_angular_acceleration>
+            <min_angular_acceleration>-1.8</min_angular_acceleration>
             <topic>cmd_vel_gz</topic>
             <odom_topic>odom</odom_topic>

Commit message: refactor(nav2): align velocity limits and costmap with real hardware
- Scale MPPI/velocity_smoother/behavior_server limits to the measured
  wheel speed (13 rad/s): vx_max=0.52 m/s, wz_max=2.0 rad/s, with
  matching accelerations; fix wheel_separation (0.26m) and
  max_wheel_velocity (13 rad/s) docs to match
- Fix robot_base_frame (base_link -> base_footprint) across costmaps,
  bt_navigator and behavior_server
- Replace local_costmap voxel_layer with a 2D obstacle_layer and tune
  inflation (cost_scaling_factor 6.0, inflation_radius 0.15) so the
  planner stops avoiding passable narrow corridors
- Enable TwirlingCritic and lower PathAlignCritic weight for more
  flexible path following
- Add a 0.20m emergency-stop circle to collision_monitor
- Remove unused docking_server and loopback_simulator (no dock
  configured)
- Ignore *.tmp files

File: pizibot_description/urdf/dimensions.xacro (robot description, xacro)
@@ -12,6 +12,6 @@
     <xacro:property name="wheel_y_offset" value="0.01969" />
     <xacro:property name="wheel_friction" value="1.0" />
-    <!-- Max wheel velocity property in rad/s (13.0 rad/s ≈ 124.1 RPM, matches WHEEL_CMD_MAX_RADS) -->
-    <xacro:property name="max_wheel_velocity" value="13.0" />
+    <!-- Max wheel velocity property in rad/s (10.0 rad/s ≈ 95.5 RPM, matches WHEEL_CMD_MAX_RADS) -->
+    <xacro:property name="max_wheel_velocity" value="10.0" />
     <!-- Max wheel effort in Nm -->
     <xacro:property name="max_wheel_effort" value="40" />
